Commit message: Final Commit, everything tested and works

File: urdf/slam_bot.xacro (robot description, xacro)
@@ -22,5 +22,5 @@
       <origin xyz="0 0 0" rpy=" 0 0 0"/>
       <geometry>
-        <box size=".4 .2 .1"/>
+        <box size=".4 .4 .1"/>
       </geometry>
     </collision>
@@ -28,5 +28,5 @@
       <origin xyz="0 0 0" rpy=" 0 0 0"/>
       <geometry>
-        <box size=".4 .2 .1"/>
+        <box size=".4 .4 .1"/>
       </geometry>
     <material name="orange"/>
@@ -101,5 +101,5 @@
   </link>
   <joint type="continuous" name="left_wheel_hinge">
-    <origin xyz="0 0.15 0" rpy="0 0 0"/>
+    <origin xyz="0 0.25 0" rpy="0 0 0"/>
     <child link="left_wheel"/>
     <parent link="chassis"/>
@@ -132,5 +132,5 @@
   </link>
   <joint type="continuous" name="right_wheel_hinge">
-    <origin xyz="0 -0.15 0" rpy="0 0 0"/>
+    <origin xyz="0 -0.25 0" rpy="0 0 0"/>
     <child link="right_wheel"/>
     <parent link="chassis"/>
@@ -168,9 +168,9 @@
     <parent link="chassis"/>
   </joint>
-    <joint type="fixed" name="camera_joint">
-    <origin xyz="0 0 0" rpy="0 0 0"/>
-    <child link="camera_rgbd_frame"/>
-    <parent link="camera"/>
-  </joint>
+ <joint name="camera_joint" type="fixed">
+        <origin xyz="0 0 0" rpy="-1.5707 0 -1.5707"/>
+        <parent link="camera"/>
+        <child link="camera_rgbd_frame"/>
+    </joint>
 <link name = "camera_rgbd_frame"/>
     <!-- Laser Rangefinder -->
@@ -191,5 +191,5 @@
       </geometry>
     </collision>
-    <visual name='camera_visual'>
+    <visual name='hokuyo_visual'>
       <origin xyz="0.0 0 0.0" rpy=" 0 0 0"/>
       <geometry>
@@ -199,5 +199,5 @@
   </link>
   <joint type="fixed" name="hokuyo_joint">
-    <origin xyz=".15 0 .1" rpy="0 0 0"/>
+    <origin xyz=".175 0 .1" rpy="0 0 0"/>
     <child link="hokuyo"/>
     <parent link="chassis"/>
